File: minrc-ref/minrc-ref_pcb/minrc-ref.kicad_pcb (KiCad board)
At the start: 2 copper layers, 1 part, among them U1 ESP32S3

Commit message: workshop
Parts:
- added J1: Conn_01x04, pcblearning:PM08_stepper_motor, B.Cu at (149.7, 101.5)
- added U2: DRV8837, Package_SON:WSON-8-1EP_2x2mm_P0.5mm_EP0.9x1.6mm, F.Cu at (139.2, 98.5)
- added U3: DRV8837, Package_SON:WSON-8-1EP_2x2mm_P0.5mm_EP0.9x1.6mm, F.Cu at (139.4, 105.0)
- U1: footprint pcblearning:esp32s3-supermini -> pcblearning:ESP32-S3-SUPERMINI
- moved U1 49.0 mm to (120.5, 90.4)
Connections:
- U1 pad 12: unconnected-(U1-GPIO10-Pad12) -> Net-(U1-GPIO10)
- U1 pad 13: unconnected-(U1-GPIO11-Pad13) -> Net-(U1-GPIO11)
- U1 pad 14: unconnected-(U1-GPIO12-Pad14) -> Net-(U1-GPIO12)
- U1 pad 15: unconnected-(U1-GPIO13-Pad15) -> Net-(U1-GPIO13)
- U1 pad 17: unconnected-(U1-GND-Pad17) -> GND
Routing:
- net Net-(U1-GPIO12): track 0.00 -> 11.1 mm
- net Net-(U1-GPIO11): track 0.00 -> 10.8 mm
- net Net-(U1-GPIO10): track 0.00 -> 10.7 mm
- net Net-(J1-Pin_3): track 0.00 -> 10.3 mm
- net Net-(J1-Pin_2): track 0.00 -> 10.3 mm
- net Net-(U1-GPIO13): track 0.00 -> 10.2 mm
- net Net-(J1-Pin_4): track 0.00 -> 9.92 mm
- net Net-(J1-Pin_1): track 0.00 -> 9.84 mm
- added copper zone on F.Cu, net GND
Other:
- board outline added: 45.8 x 29.4 mm
