File: minrc-ref/minrc-ref_pcb/minrc-ref.kicad_sch (KiCad schematic)
At the start: 1 part, among them U1 ESP32S3

Commit message: workshop
Parts:
- removed U1: ESP32S3, pcblearning:esp32s3-supermini, symbol pcblearning:esp32s3-supermini
- added J1: Conn_01x04, pcblearning:PM08_stepper_motor, symbol Connector_Generic:Conn_01x04
- added U1: ESP32S3, pcblearning:ESP32-S3-SUPERMINI, symbol pcblearning:ESP32-S3-SUPERMINI
- added U2, U3: DRV8837, Package_SON:WSON-8-1EP_2x2mm_P0.5mm_EP0.9x1.6mm, symbol Driver_Motor:DRV8837
Connections:
- new net: J1.2 (Pin_2), U2.2 (OUT1)
- new net: J1.1 (Pin_1), U2.3 (OUT2)
- new net: U1.15 (GPIO13), U2.5 (IN2)
- new net: U1.14 (GPIO12), U2.6 (IN1)
- new net: J1.4 (Pin_4), U3.2 (OUT1)
- new net: J1.3 (Pin_3), U3.3 (OUT2)
- new net: U1.13 (GPIO11), U3.5 (IN2)
- new net: U1.12 (GPIO10), U3.6 (IN1)
- new net GND: U1.17 (GND), U2.4 (GND), U2.9 (GND), U3.4 (GND), U3.9 (GND)
